Commit message: xacro

File: urdf/simple.xacro (robot description, xacro)
@@ -1,4 +1,5 @@
 <?xml version="1.0"?>
-<robot name="simple_robot">
+<robot name="simple_robot" xmlns:xacro="http://ros.org/wiki/xacro">
+  <xacro:include filename="./materials.xacro" />
   <link name="base_link">
     <visual>
@@ -8,4 +9,5 @@
       <!-- set visual origin in the coordinate frame of link -->
       <origin xyz="0 0 0.2"/>
+      <material name="blue"/>
     </visual>
   </link>
@@ -15,4 +17,5 @@
         <box size="0.3 0.3 0.6"/>
       </geometry>
+      <material name="orange"/>
     </visual>
   </link>

Commit message: xacro simple.xacro > simple.urdf
Run gazebo and insert model (Add path,

browse the simple directory
and gazebo will show you the model "simple")

File: urdf/simple.xacro (robot description, xacro)
@@ -2,4 +2,17 @@
 <robot name="simple_robot" xmlns:xacro="http://ros.org/wiki/xacro">
   <xacro:include filename="./materials.xacro" />
+  <xacro:macro name="default_inertial" params="mass">
+    <inertial>
+      <mass value="${mass}">${mass}</mass>
+      <inertia ixx="1.0" ixy="0.0" ixz="0.0" iyy="1.0" iyz="0.0" izz="1.0">
+          <ixx>1</ixx>
+          <ixy>0</ixy>
+          <ixz>0</ixz>
+          <iyy>1</iyy>
+          <iyz>0</iyz>
+          <izz>1</izz>
+      </inertia>
+    </inertial>
+  </xacro:macro>
   <link name="base_link">
     <visual>
@@ -11,4 +24,12 @@
       <material name="blue"/>
     </visual>
+    <collision>
+      <geometry>
+        <cylinder length="0.4" radius="0.4"/>
+      </geometry>
+      <!-- set visual origin in the coordinate frame of link -->
+      <origin xyz="0 0 0.2"/>
+    </collision>
+    <xacro:default_inertial mass="1"/>
   </link>
   <link name="body_link">
@@ -19,4 +40,10 @@
       <material name="orange"/>
     </visual>
+    <collision>
+      <geometry>
+        <box size="0.3 0.3 0.6"/>
+      </geometry>
+    </collision>
+    <xacro:default_inertial mass="1"/>
   </link>
   <joint name="base_body_joint" type="continuous">
@@ -26,3 +53,4 @@
     <axis xyz="0 0 1"/>
   </joint>
+  <xacro:include filename="./simple.gazebo" />
 </robot>
